File: digital.kicad_sch (KiCad schematic)
At the start: 33 parts

Commit message: WIP
Parts:
- gave numbers to parts that had none: 33
Connections:
- net SCL: now also U2.17 (SDA); no longer U2.18 (SCL)
- net SDA: now also U2.18 (SCL); no longer U2.17 (SDA)
Other:
- moved on the sheet: C1, C10, C11, C12, C13, C14, C2, C3, C4, C5, C6, C7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

Commit message: WIP
Parts:
- removed R4: 10K, Resistor_SMD:R_0805_2012Metric, symbol Device:R
- C11, C13, C14, C2, C4, C7: footprint Capacitor_SMD:C_0805_2012Metric -> Capacitor_SMD:C_0603_1608Metric
- C9: value 10uF -> 100nF; footprint Capacitor_SMD:C_0805_2012Metric -> Capacitor_SMD:C_0603_1608Metric
- D1: footprint Resistor_SMD:R_0805_2012Metric -> LED_SMD:LED_0805_2012Metric
- J4: renamed from J3; footprint Resistor_SMD:R_0805_2012Metric -> Connector_PinHeader_2.54mm:PinHeader_1x02_P2.54mm_Vertical
Connections:
- net at R1.1, U2.1 (XSMT): now also U2.24 (MODE2), U2.32 (ADR1)
Other:
- moved on the sheet: R1
Changed lines of the file:
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@@
   (junction (at 207.01 96.52) (diameter 0) (color 0 0 0 0)
+  )
+  (junction (at 92.71 36.83) (diameter 0) (color 0 0 0 0)
   )
   (junction (at 71.12 54.61) (diameter 0) (color 0 0 0 0)
@@
     (stroke (width 0) (type default) (color 0 0 0 0))
   )
+  (wire (pts (xy 92.71 36.83) (xy 92.71 49.53))
+    (stroke (width 0) (type default) (color 0 0 0 0))
+  )
   (wire (pts (xy 83.82 69.85) (xy 95.25 69.85))
     (stroke (width 0) (type default) (color 0 0 0 0))
@@
     (stroke (width 0) (type default) (color 0 0 0 0))
   )
+  (wire (pts (xy 135.89 36.83) (xy 92.71 36.83))
+    (stroke (width 0) (type default) (color 0 0 0 0))
+  )
   (wire (pts (xy 135.89 72.39) (xy 135.89 74.93))
     (stroke (width 0) (type default) (color 0 0 0 0))
@@
     (stroke (width 0) (type default) (color 0 0 0 0))
   )
-  (wire (pts (xy 135.89 38.1) (xy 135.89 40.64))
-    (stroke (width 0) (type default) (color 0 0 0 0))
-  )
   (wire (pts (xy 71.12 44.45) (xy 71.12 41.91))
     (stroke (width 0) (type default) (color 0 0 0 0))
@@
     (stroke (width 0) (type default) (color 0 0 0 0))
   )
-  (wire (pts (xy 135.89 48.26) (xy 135.89 49.53))
+  (wire (pts (xy 135.89 36.83) (xy 135.89 49.53))
     (stroke (width 0) (type default) (color 0 0 0 0))
   )
@@
     (stroke (width 0) (type default) (color 0 0 0 0))
   )
-  (wire (pts (xy 92.71 38.1) (xy 92.71 40.64))
+  (wire (pts (xy 92.71 24.13) (xy 92.71 26.67))
     (stroke (width 0) (type default) (color 0 0 0 0))
   )
@@
     (stroke (width 0) (type default) (color 0 0 0 0))
   )
-  (wire (pts (xy 92.71 48.26) (xy 92.71 49.53))
+  (wire (pts (xy 92.71 34.29) (xy 92.71 36.83))
     (stroke (width 0) (type default) (color 0 0 0 0))
   )
@@
     (effects (font (size 1.27 1.27)) (justify left bottom))
   )
-  (label "DVDD" (at 135.89 38.1 90)
-    (effects (font (size 1.27 1.27)) (justify left bottom))
-  )
   (label "CLK" (at 137.16 64.77 0)
     (effects (font (size 1.27 1.27)) (justify left bottom))
@@
   (label "GPIO6" (at 204.47 55.88 180)
     (effects (font (size 1.27 1.27)) (justify right bottom))
-  )
-  (label "AVDD" (at 72.39 82.55 180)
-    (effects (font (size 1.27 1.27)) (justify right bottom))
-  )
-  (label "DVDD" (at 92.71 38.1 90)
-    (effects (font (size 1.27 1.27)) (justify left bottom))
   )
   (label "DVDD" (at 142.24 157.48 0)
@@
     )
   )
+  (global_label "AVDD" (shape input) (at 72.39 82.55 180) (fields_autoplaced)
+    (effects (font (size 1.27 1.27)) (justify right))
+    (property "Intersheet References" "${INTERSHEET_REFS}" (id 0) (at 65.2598 82.4706 0)
+      (effects (font (size 1.27 1.27)) (justify right) hide)
+    )
+  )
   (global_label "DVDD" (shape input) (at 29.21 57.15 180) (fields_autoplaced)
     (effects (font (size 1.27 1.27)) (justify right))
@@
     )
   )
+  (global_label "DVDD" (shape input) (at 92.71 24.13 90) (fields_autoplaced)
+    (effects (font (size 1.27 1.27)) (justify left))
+    (property "Intersheet References" "${INTERSHEET_REFS}" (id 0) (at 92.7894 16.8183 90)
+      (effects (font (size 1.27 1.27)) (justify left) hide)
+    )
+  )
   (hierarchical_label "ID_SC" (shape bidirectional) (at 123.19 154.94 0)
     (effects (font (size 1.27 1.27)) (justify left))
@@
       (effects (font (size 1.27 1.27)) (justify right))
     )
-    (property "Footprint" "Capacitor_SMD:C_0805_2012Metric" (id 2) (at 195.2752 85.09 0)
+    (property "Footprint" "Capacitor_SMD:C_0603_1608Metric" (id 2) (at 195.2752 85.09 0)
       (effects (font (size 1.27 1.27)) hide)
     )
@@
       (effects (font (size 1.27 1.27)) (justify left))
     )
-    (property "Value" "10uF" (id 1) (at 83.82 90.1699 0)
-      (effects (font (size 1.27 1.27)) (justify left))
-    )
-    (property "Footprint" "Capacitor_SMD:C_0805_2012Metric" (id 2) (at 80.9752 92.71 0)
+    (property "Value" "100nF" (id 1) (at 83.82 90.1699 0)
+      (effects (font (size 1.27 1.27)) (justify left))
+    )
+    (property "Footprint" "Capacitor_SMD:C_0603_1608Metric" (id 2) (at 80.9752 92.71 0)
       (effects (font (size 1.27 1.27)) hide)
     )
@@
       (effects (font (size 1.27 1.27)) (justify left))
     )
-    (property "Footprint" "Capacitor_SMD:C_0805_2012Metric" (id 2) (at 67.0052 67.31 0)
+    (property "Footprint" "Capacitor_SMD:C_0603_1608Metric" (id 2) (at 67.0052 67.31 0)
       (effects (font (size 1.27 1.27)) hide)
     )
@@
       (effects (font (size 1.27 1.27)) (justify left))
     )
-    (property "Footprint" "Capacitor_SMD:C_0805_2012Metric" (id 2) (at 87.9348 151.13 0)
+    (property "Footprint" "Capacitor_SMD:C_0603_1608Metric" (id 2) (at 87.9348 151.13 0)
       (effects (font (size 1.27 1.27)) hide)
     )
@@
   (symbol (lib_id "Connector_Generic:Conn_02x01") (at 127 165.1 270) (unit 1)
     (in_bom yes) (on_board yes) (fields_autoplaced)
-    (property "Reference" "J3" (id 0) (at 129.54 165.0999 90)
+    (property "Reference" "J4" (id 0) (at 129.54 165.0999 90)
       (effects (font (size 1.27 1.27)) (justify left))
     )
@@
       (effects (font (size 1.27 1.27)) (justify left))
     )
-    (property "Footprint" "Resistor_SMD:R_0805_2012Metric" (id 2) (at 127 165.1 0)
+    (property "Footprint" "Connector_PinHeader_2.54mm:PinHeader_1x02_P2.54mm_Vertical" (id 2) (at 127 165.1 0)
       (effects (font (size 1.27 1.27)) hide)
     )
@@
       (effects (font (size 1.27 1.27)) (justify left))
     )
-    (property "Footprint" "Capacitor_SMD:C_0805_2012Metric" (id 2) (at 77.1652 52.07 0)
+    (property "Footprint" "Capacitor_SMD:C_0603_1608Metric" (id 2) (at 77.1652 52.07 0)
       (effects (font (size 1.27 1.27)) hide)
     )
@@
     (property "Reference" "D1" (id 0) (at 143.8275 72.39 0))
     (property "Value" "LED" (id 1) (at 143.8275 74.93 0))
-    (property "Footprint" "Resistor_SMD:R_0805_2012Metric" (id 2) (at 142.24 80.01 0)
+    (property "Footprint" "LED_SMD:LED_0805_2012Metric" (id 2) (at 142.24 80.01 0)
       (effects (font (size 1.27 1.27)) hide)
     )
@@
       (effects (font (size 1.27 1.27)) (justify left))
     )
-    (property "Footprint" "Capacitor_SMD:C_0805_2012Metric" (id 2) (at 40.3352 64.77 0)
+    (property "Footprint" "Capacitor_SMD:C_0603_1608Metric" (id 2) (at 40.3352 64.77 0)
       (effects (font (size 1.27 1.27)) hide)
     )
@@
     )
     (pin "1")
-  )
-  (symbol (lib_id "Device:R") (at 135.89 44.45 180) (unit 1)
-    (in_bom yes) (on_board yes) (fields_autoplaced)
-    (property "Reference" "R4" (id 0) (at 138.43 43.1799 0)
-      (effects (font (size 1.27 1.27)) (justify right))
-    )
-    (property "Value" "10K" (id 1) (at 138.43 45.7199 0)
-      (effects (font (size 1.27 1.27)) (justify right))
-    )
-    (property "Footprint" "Resistor_SMD:R_0805_2012Metric" (id 2) (at 137.668 44.45 90)
-      (effects (font (size 1.27 1.27)) hide)
-    )
-    (property "Datasheet" "~" (id 3) (at 135.89 44.45 0)
-      (effects (font (size 1.27 1.27)) hide)
-    )
-    (pin "1")
-    (pin "2")
   )
   (symbol (lib_id "Device:R") (at 151.13 80.01 90) (unit 1)
@@
       (effects (font (size 1.27 1.27)) (justify right))
     )
-    (property "Footprint" "Capacitor_SMD:C_0805_2012Metric" (id 2) (at 195.2752 50.8 0)
+    (property "Footprint" "Capacitor_SMD:C_0603_1608Metric" (id 2) (at 195.2752 50.8 0)
       (effects (font (size 1.27 1.27)) hide)
     )
@@
     (pin "2")
   )
-  (symbol (lib_id "Device:R") (at 92.71 44.45 180) (unit 1)
-    (in_bom yes) (on_board yes) (fields_autoplaced)
-    (property "Reference" "R1" (id 0) (at 95.25 43.1799 0)
+  (symbol (lib_id "Device:R") (at 92.71 30.48 180) (unit 1)
+    (in_bom yes) (on_board yes) (fields_autoplaced)
+    (property "Reference" "R1" (id 0) (at 95.25 29.2099 0)
       (effects (font (size 1.27 1.27)) (justify right))
     )
-    (property "Value" "10K" (id 1) (at 95.25 45.7199 0)
+    (property "Value" "10K" (id 1) (at 95.25 31.7499 0)
       (effects (font (size 1.27 1.27)) (justify right))
     )
-    (property "Footprint" "Resistor_SMD:R_0805_2012Metric" (id 2) (at 94.488 44.45 90)
-      (effects (font (size 1.27 1.27)) hide)
-    )
-    (property "Datasheet" "~" (id 3) (at 92.71 44.45 0)
-      (effects (font (size 1.27 1.27)) hide)
-    )
+    (property "Footprint" "Resistor_SMD:R_0805_2012Metric" (id 2) (at 94.488 30.48 90)
+      (effects (font (size 1.27 1.27)) hide)
+    )
+    (property "Datasheet" "~" (id 3) (at 92.71 30.48 0)
+      (effects (font (size 1.27 1.27)) hide)
+    )
