File: psu.kicad_sch (KiCad schematic)
At the start: 16 parts

Commit message: WIP
Parts:
- C17, C18, C19, C20: renamed from C?; footprint Capacitor_SMD:C_0805_2012Metric -> Capacitor_SMD:C_1206_3216Metric
- gave numbers to parts that had none: 12
Other:
- note added: "ZVD for protecting Raspberry Pi from accidentally powering amplifier."
- moved on the sheet: C15, C16, C19, C20, C21, L1, Q1, R14, R15, U6

Commit message: WIP
Parts:
- C16: footprint Capacitor_SMD:C_0805_2012Metric -> Capacitor_SMD:C_0603_1608Metric
Changed lines of the file:
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@@
   (junction (at 210.82 57.15) (diameter 0) (color 0 0 0 0)
   )
+  (junction (at 78.74 71.12) (diameter 0) (color 0 0 0 0)
+  )
   (junction (at 213.36 78.74) (diameter 0) (color 0 0 0 0)
   )
@@
     (stroke (width 0) (type default) (color 0 0 0 0))
   )
+  (polyline (pts (xy 195.58 35.56) (xy 243.84 35.56))
+    (stroke (width 0) (type default) (color 0 0 0 0))
+  )
+  (polyline (pts (xy 243.84 105.41) (xy 195.58 105.41))
+    (stroke (width 0) (type default) (color 0 0 0 0))
+  )
   (wire (pts (xy 224.79 53.34) (xy 228.6 53.34))
     (stroke (width 0) (type default) (color 0 0 0 0))
@@
     (stroke (width 0) (type default) (color 0 0 0 0))
   )
-  (wire (pts (xy 78.74 62.23) (xy 78.74 72.39))
-    (stroke (width 0) (type default) (color 0 0 0 0))
-  )
   (wire (pts (xy 115.57 57.15) (xy 118.11 57.15))
     (stroke (width 0) (type default) (color 0 0 0 0))
   )
+  (wire (pts (xy 78.74 62.23) (xy 78.74 71.12))
+    (stroke (width 0) (type default) (color 0 0 0 0))
+  )
   (wire (pts (xy 88.9 57.15) (xy 96.52 57.15))
     (stroke (width 0) (type default) (color 0 0 0 0))
@@
     (stroke (width 0) (type default) (color 0 0 0 0))
   )
+  (polyline (pts (xy 243.84 35.56) (xy 243.84 105.41))
+    (stroke (width 0) (type default) (color 0 0 0 0))
+  )
   (wire (pts (xy 222.25 73.66) (xy 222.25 78.74))
     (stroke (width 0) (type default) (color 0 0 0 0))
@@
     (stroke (width 0) (type default) (color 0 0 0 0))
   )
+  (wire (pts (xy 78.74 71.12) (xy 78.74 72.39))
+    (stroke (width 0) (type default) (color 0 0 0 0))
+  )
   (wire (pts (xy 88.9 163.83) (xy 88.9 166.37))
     (stroke (width 0) (type default) (color 0 0 0 0))
   )
   (wire (pts (xy 54.61 52.07) (xy 63.5 52.07))
+    (stroke (width 0) (type default) (color 0 0 0 0))
+  )
+  (polyline (pts (xy 195.58 35.56) (xy 195.58 105.41))
     (stroke (width 0) (type default) (color 0 0 0 0))
   )
@@
   (symbol (lib_id "power:PWR_FLAG") (at 115.57 55.88 0) (unit 1)
     (in_bom yes) (on_board yes)
-    (property "Reference" "#FLG02" (id 0) (at 115.57 53.975 0)
+    (property "Reference" "#FLG03" (id 0) (at 115.57 53.975 0)
       (effects (font (size 1.27 1.27)) hide)
     )
@@
     (pin "1")
     (pin "2")
+  )
+  (symbol (lib_id "power:PWR_FLAG") (at 78.74 71.12 90) (unit 1)
+    (in_bom yes) (on_board yes)
+    (property "Reference" "#FLG02" (id 0) (at 76.835 71.12 0)
+      (effects (font (size 1.27 1.27)) hide)
+    )
+    (property "Value" "PWR_FLAG" (id 1) (at 74.93 71.12 90)
+      (effects (font (size 1.27 1.27)) (justify left))
+    )
+    (property "Footprint" "" (id 2) (at 78.74 71.12 0)
+      (effects (font (size 1.27 1.27)) hide)
+    )
+    (property "Datasheet" "~" (id 3) (at 78.74 71.12 0)
+      (effects (font (size 1.27 1.27)) hide)
+    )
+    (pin "1")
   )
   (symbol (lib_id "Etnolit:DMMT5401") (at 219.71 67.31 0) (unit 1)
@@
       (effects (font (size 1.27 1.27)) (justify left))
     )
-    (property "Footprint" "Capacitor_SMD:C_0805_2012Metric" (id 2) (at 55.5752 67.31 0)
-      (effects (font (size 1.27 1.27)) hide)
-    )
+    (property "Footprint" "Capacitor_SMD:C_0603_1608Metric" (id 2) (at 55.5752 67.31 0)
+      (effects (font (size 1.27 1.27)) hide)
+    )

Commit message: WIP
Parts:
- removed U4, U5: LM1117-3.3, Package_TO_SOT_SMD:SOT-223-3_TabPin2, symbol Regulator_Linear:LM1117-3.3
- added U4, U5: NCP163ASN330T1G, Package_TO_SOT_SMD:SOT-23-5, symbol Etnolit:NCP163
- C17, C18, C19, C20: footprint Capacitor_SMD:C_1206_3216Metric -> Capacitor_SMD:C_0805_2012Metric; Type tantalum -> (none)
Connections:
- net 5V: now also U4.1 (IN), U4.3 (EN), U5.1 (IN), U5.3 (EN)
- net AVDD: now also U5.5 (OUT)
- net DVDD: now also U4.5 (OUT)
- net GND: now also U4.2 (GND), U4.4 (NC), U5.2 (GND), U5.4 (NC)
Changed lines of the file:
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@@
   (junction (at 217.17 78.74) (diameter 0) (color 0 0 0 0)
   )
+  (junction (at 66.04 153.67) (diameter 0) (color 0 0 0 0)
+  )
   (junction (at 115.57 57.15) (diameter 0) (color 0 0 0 0)
   )
   (junction (at 54.61 52.07) (diameter 0) (color 0 0 0 0)
   )
+  (junction (at 66.04 110.49) (diameter 0) (color 0 0 0 0)
+  )
   (junction (at 210.82 57.15) (diameter 0) (color 0 0 0 0)
   )
@@
     (stroke (width 0) (type default) (color 0 0 0 0))
   )
-  (wire (pts (xy 59.69 153.67) (xy 68.58 153.67))
+  (wire (pts (xy 59.69 153.67) (xy 66.04 153.67))
     (stroke (width 0) (type default) (color 0 0 0 0))
   )
@@
     (stroke (width 0) (type default) (color 0 0 0 0))
   )
+  (wire (pts (xy 66.04 156.21) (xy 66.04 153.67))
+    (stroke (width 0) (type default) (color 0 0 0 0))
+  )
   (wire (pts (xy 88.9 153.67) (xy 91.44 153.67))
     (stroke (width 0) (type default) (color 0 0 0 0))
@@
     (stroke (width 0) (type default) (color 0 0 0 0))
   )
+  (wire (pts (xy 66.04 113.03) (xy 66.04 110.49))
+    (stroke (width 0) (type default) (color 0 0 0 0))
+  )
   (wire (pts (xy 226.06 76.2) (xy 226.06 80.01))
     (stroke (width 0) (type default) (color 0 0 0 0))
   )
+  (wire (pts (xy 68.58 156.21) (xy 66.04 156.21))
+    (stroke (width 0) (type default) (color 0 0 0 0))
+  )
+  (wire (pts (xy 66.04 153.67) (xy 68.58 153.67))
+    (stroke (width 0) (type default) (color 0 0 0 0))
+  )
   (polyline (pts (xy 195.58 35.56) (xy 243.84 35.56))
     (stroke (width 0) (type default) (color 0 0 0 0))
@@
     (stroke (width 0) (type default) (color 0 0 0 0))
   )
-  (wire (pts (xy 76.2 161.29) (xy 76.2 166.37))
-    (stroke (width 0) (type default) (color 0 0 0 0))
-  )
   (wire (pts (xy 226.06 60.96) (xy 226.06 57.15))
     (stroke (width 0) (type default) (color 0 0 0 0))
@@
     (stroke (width 0) (type default) (color 0 0 0 0))
   )
+  (wire (pts (xy 76.2 119.38) (xy 76.2 123.19))
+    (stroke (width 0) (type default) (color 0 0 0 0))
+  )
   (wire (pts (xy 115.57 57.15) (xy 118.11 57.15))
     (stroke (width 0) (type default) (color 0 0 0 0))
@@
     (stroke (width 0) (type default) (color 0 0 0 0))
   )
-  (wire (pts (xy 59.69 110.49) (xy 68.58 110.49))
+  (wire (pts (xy 59.69 110.49) (xy 66.04 110.49))
     (stroke (width 0) (type default) (color 0 0 0 0))
   )
@@
     (stroke (width 0) (type default) (color 0 0 0 0))
   )
+  (wire (pts (xy 66.04 110.49) (xy 68.58 110.49))
+    (stroke (width 0) (type default) (color 0 0 0 0))
+  )
   (wire (pts (xy 104.14 57.15) (xy 111.76 57.15))
     (stroke (width 0) (type default) (color 0 0 0 0))
@@
     (stroke (width 0) (type default) (color 0 0 0 0))
   )
-  (wire (pts (xy 76.2 118.11) (xy 76.2 123.19))
+  (wire (pts (xy 76.2 162.56) (xy 76.2 166.37))
     (stroke (width 0) (type default) (color 0 0 0 0))
   )
@@
   )
   (wire (pts (xy 88.9 163.83) (xy 88.9 166.37))
+    (stroke (width 0) (type default) (color 0 0 0 0))
+  )
+  (wire (pts (xy 68.58 113.03) (xy 66.04 113.03))
     (stroke (width 0) (type default) (color 0 0 0 0))
   )
@@
     (pin "1")
   )
-  (symbol (lib_id "Regulator_Linear:LM1117-3.3") (at 76.2 110.49 0) (unit 1)
-    (in_bom yes) (on_board yes) (fields_autoplaced)
-    (property "Reference" "U4" (id 0) (at 76.2 102.87 0))
-    (property "Value" "LM1117-3.3" (id 1) (at 76.2 105.41 0))
-    (property "Footprint" "Package_TO_SOT_SMD:SOT-223-3_TabPin2" (id 2) (at 76.2 110.49 0)
-      (effects (font (size 1.27 1.27)) hide)
-    )
-    (property "Datasheet" "http://www.ti.com/lit/ds/symlink/lm1117.pdf" (id 3) (at 76.2 110.49 0)
-      (effects (font (size 1.27 1.27)) hide)
-    )
-    (pin "1")
-    (pin "2")
-    (pin "3")
-  )
   (symbol (lib_id "power:GND") (at 111.76 72.39 0) (unit 1)
     (in_bom yes) (on_board yes) (fields_autoplaced)
@@
       (effects (font (size 1.27 1.27)) (justify left))
     )
-    (property "Footprint" "Capacitor_SMD:C_1206_3216Metric" (id 2) (at 89.8652 120.65 0)
+    (property "Footprint" "Capacitor_SMD:C_0805_2012Metric" (id 2) (at 89.8652 120.65 0)
       (effects (font (size 1.27 1.27)) hide)
     )
     (property "Datasheet" "~" (id 3) (at 88.9 116.84 0)
       (effects (font (size 1.27 1.27)) hide)
-    )
-    (property "Type" "tantalum" (id 4) (at 92.71 120.65 0)
-      (effects (font (size 1.27 1.27)) (justify left))
     )
     (pin "1")
@@
       (effects (font (size 1.27 1.27)) (justify left))
     )
-    (property "Footprint" "Capacitor_SMD:C_1206_3216Metric" (id 2) (at 89.8652 163.83 0)
+    (property "Footprint" "Capacitor_SMD:C_0805_2012Metric" (id 2) (at 89.8652 163.83 0)
       (effects (font (size 1.27 1.27)) hide)
     )
@@
       (effects (font (size 1.27 1.27)) hide)
     )
-    (property "Type" "tantalum" (id 4) (at 92.71 163.83 0)
-      (effects (font (size 1.27 1.27)) (justify left))
-    )
-    (pin "1")
-    (pin "2")
-  )
-  (symbol (lib_id "Regulator_Linear:LM1117-3.3") (at 76.2 153.67 0) (unit 1)
-    (in_bom yes) (on_board yes) (fields_autoplaced)
-    (property "Reference" "U5" (id 0) (at 76.2 146.05 0))
-    (property "Value" "LM1117-3.3" (id 1) (at 76.2 148.59 0))
-    (property "Footprint" "Package_TO_SOT_SMD:SOT-223-3_TabPin2" (id 2) (at 76.2 153.67 0)
-      (effects (font (size 1.27 1.27)) hide)
-    )
-    (property "Datasheet" "http://www.ti.com/lit/ds/symlink/lm1117.pdf" (id 3) (at 76.2 153.67 0)
-      (effects (font (size 1.27 1.27)) hide)
-    )
-    (pin "1")
-    (pin "2")
-    (pin "3")
+    (pin "1")
+    (pin "2")
   )
   (symbol (lib_id "power:GND") (at 226.06 88.9 0) (unit 1)
@@
     (pin "1")
   )
+  (symbol (lib_id "Etnolit:NCP163") (at 76.2 156.21 0) (unit 1)
+    (in_bom yes) (on_board yes)
+    (property "Reference" "U5" (id 0) (at 76.2 148.59 0))
+    (property "Value" "NCP163ASN330T1G" (id 1) (at 76.2 151.13 0))
+    (property "Footprint" "Package_TO_SOT_SMD:SOT-23-5" (id 2) (at 76.2 156.21 0)
+      (effects (font (size 1.27 1.27)) hide)
+    )
+    (property "Datasheet" "" (id 3) (at 76.2 156.21 0)
+      (effects (font (size 1.27 1.27)) hide)
+    )
+    (pin "1")
+    (pin "2")
+    (pin "3")
+    (pin "4")
+    (pin "5")
+  )
   (symbol (lib_id "Etnolit:LM2592HV") (at 74.93 54.61 0) (unit 1)
     (in_bom yes) (on_board yes)
@@
     (pin "5")
   )
+  (symbol (lib_id "Etnolit:NCP163") (at 76.2 113.03 0) (unit 1)
+    (in_bom yes) (on_board yes)
+    (property "Reference" "U4" (id 0) (at 76.2 105.41 0))
+    (property "Value" "NCP163ASN330T1G" (id 1) (at 76.2 107.95 0))
+    (property "Footprint" "Package_TO_SOT_SMD:SOT-23-5" (id 2) (at 76.2 113.03 0)
+      (effects (font (size 1.27 1.27)) hide)
+    )
+    (property "Datasheet" "" (id 3) (at 76.2 113.03 0)
+      (effects (font (size 1.27 1.27)) hide)
+    )
+    (pin "1")
+    (pin "2")
+    (pin "3")
+    (pin "4")
+    (pin "5")
+  )
   (symbol (lib_id "power:GND") (at 88.9 166.37 0) (unit 1)
     (in_bom yes) (on_board yes) (fields_autoplaced)
@@
       (effects (font (size 1.27 1.27)) (justify left))
     )
-    (property "Footprint" "Capacitor_SMD:C_1206_3216Metric" (id 2) (at 60.6552 120.65 0)
+    (property "Footprint" "Capacitor_SMD:C_0805_2012Metric" (id 2) (at 60.6552 120.65 0)
       (effects (font (size 1.27 1.27)) hide)
     )
@@
       (effects (font (size 1.27 1.27)) hide)
     )
-    (property "Type" "tantalum" (id 4) (at 63.5 120.65 0)
-      (effects (font (size 1.27 1.27)) (justify left))
-    )
     (pin "1")
     (pin "2")
@@
       (effects (font (size 1.27 1.27)) (justify left))
     )
-    (property "Footprint" "Capacitor_SMD:C_1206_3216Metric" (id 2) (at 60.6552 163.83 0)
+    (property "Footprint" "Capacitor_SMD:C_0805_2012Metric" (id 2) (at 60.6552 163.83 0)
       (effects (font (size 1.27 1.27)) hide)
     )
@@
       (effects (font (size 1.27 1.27)) hide)
     )
-    (property "Type" "tantalum" (id 4) (at 63.5 163.83 0)
-      (effects (font (size 1.27 1.27)) (justify left))
-    )
-    (pin "1")
+    (pin "1")
