File: DesktopAMP.kicad_pcb (KiCad board)
At the start: 2 copper layers, 100 x 100 mm, 82 parts, among them J1 Conn_02x20_Odd_Even, J2 Conn_01x03, J3 Conn_01x04, J4 Conn_02x01, J5 Conn_01x03, Q1 DMG2305UX, U1 AT24CS01-STUM, U2 PCM5242, U3 LM2592HV, U4 LM1117-3.3, U5 LM1117-3.3, U6 DMMT5401, U7 LM4780, X1 22.5792MHz, X2 24.5760MHz

Commit message: WIP
Parts:
- added L2: 0.7uH, Etnolit:L_Axial_L13.25_D11.4_P13.25_Horizontal, F.Cu at (112.6, 59.5)
- added L3: 0.7uH, Etnolit:L_Axial_L13.25_D11.4_P13.25_Horizontal, F.Cu at (112.6, 95.6)
- added R31: 10R,3W, Resistor_THT:R_Axial_DIN0617_L17.0mm_D6.0mm_P20.32mm_Horizontal, F.Cu at (102.5, 59.5)
- added R32: 10R,3W, Resistor_THT:R_Axial_DIN0617_L17.0mm_D6.0mm_P20.32mm_Horizontal, F.Cu at (122.8, 95.6)
- moved R30 54.9 mm to (211.1, 80.5), turned to 0 degrees
- moved C32 52.1 mm to (210.1, 86.3), turned to 180 degrees
- moved J5 47.8 mm to (211.4, 91.4), turned to -90 degrees
- moved D3 46.5 mm to (206.7, 80.5), turned to 0 degrees
- moved R5 24.3 mm to (170.3, 132.9), turned to 90 degrees
- moved R3 22.7 mm to (182.6, 135.0), turned to 90 degrees
- moved C11 21.5 mm to (174.7, 130.3), turned to 180 degrees
- moved U1 20.5 mm to (174.7, 132.9), turned to 180 degrees
- moved R2 20.5 mm to (180.2, 135.0), turned to -90 degrees
- moved R20 19.4 mm to (190.6, 58.3)
- moved R23 17.6 mm to (187.6, 58.3)
- moved J4 14.4 mm to (173.7, 117.2), turned to 90 degrees
- moved R6 13.9 mm to (174.7, 111.4), turned to 0 degrees
- moved R8 13.9 mm to (170.7, 110.2)
- moved C1 13.1 mm to (182.9, 104.6)
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Connections:
- R25 pad 2: /Analog/L_{out}+ -> Net-(L2-Pad1)
- R26 pad 2: /Analog/R_{out}+ -> Net-(L3-Pad2)
- R28 pad 2: /Analog/L_{out}+ -> Net-(L2-Pad1)
- R29 pad 2: /Analog/R_{out}+ -> Net-(L3-Pad2)
- U7 pad 25: /Analog/R_{out}+ -> Net-(L3-Pad2)
- U7 pad 7: /Analog/L_{out}+ -> Net-(L2-Pad1)
Routing:
- net GND: track 614.6 -> 703.6 mm
- net Net-(L3-Pad2): track 0.00 -> 76.0 mm
- net /Analog/R_{out}+: track 79.4 -> 23.4 mm
- net Net-(L2-Pad1): track 0.00 -> 51.0 mm
- net /Analog/L_{out}+: track 60.1 -> 23.3 mm
- net DVDD: track 121.1 -> 91.7 mm, vias 10 -> 9
- net Net-(C23-Pad1): track 3.43 -> 29.7 mm
- net Net-(C22-Pad2): track 3.43 -> 28.5 mm
- net Net-(C23-Pad2): track 3.36 -> 26.6 mm, vias 0 -> 2
- net VEE: track 112.5 -> 91.2 mm
- net /Digital/ID_SC: track 21.7 -> 3.76 mm, vias 2 -> 0
- net /Digital/SDA: track 57.3 -> 41.6 mm, vias 0 -> 2
- net /Digital/ID_SD: track 14.4 -> 0.00 mm, vias 2 -> 0
- net /Digital/BCK: track 34.5 -> 21.0 mm
- net Net-(J4-Pad1): track 10.9 -> 0.00 mm
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- added copper zone on B.Cu, net VEE
Other:
- board text added: "Etnolit - 2002"

Commit message: WIP
Parts:
- C17, C18, C19, C20: footprint Capacitor_SMD:C_1206_3216Metric -> Capacitor_SMD:C_0805_2012Metric
- U4, U5: value LM1117-3.3 -> NCP163; footprint Package_TO_SOT_SMD:SOT-223-3_TabPin2 -> Package_TO_SOT_SMD:SOT-23-5
- moved C32 96.5 mm to (119.6, 52.7), turned to -90 degrees
- moved R30 90.2 mm to (125.6, 51.6)
- moved J5 86.9 mm to (131.6, 57.1), turned to 180 degrees
- moved D3 84.9 mm to (125.6, 55.2), turned to 180 degrees
- moved C20 33.5 mm to (163.5, 133.0), turned to 0 degrees
- moved U5 26.8 mm to (163.5, 136.6), turned to 90 degrees
- moved J4 22.8 mm to (196.5, 116.5), turned to 180 degrees
- moved C18 19.8 mm to (163.5, 140.4), turned to 0 degrees
- moved R29 19.4 mm to (102.3, 94.9), turned to 0 degrees
- moved R28 19.4 mm to (102.3, 60.1), turned to 0 degrees
- moved R31 19.2 mm to (113.7, 75.0), turned to 45 degrees
- moved C25 14.7 mm to (102.3, 91.0), turned to 0 degrees
- moved L3 11.8 mm to (120.9, 87.2), turned to -45 degrees
- moved L2 11.7 mm to (120.9, 67.8), turned to -135 degrees
- moved R5 11.1 mm to (175.3, 142.8), turned to 180 degrees
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Connections:
- U4 pad 1: GND -> /Power/5V
- U4 pad 2: DVDD -> GND
- U5 pad 1: GND -> /Power/5V
- U5 pad 2: AVDD -> GND
Routing:
- net DVDD: track 91.7 -> 141.9 mm, vias 9 -> 5
- net GND: track 703.6 -> 751.3 mm, vias 68 -> 72
- net AVDD: track 79.9 -> 125.8 mm, vias 8 -> 4
- net Net-(J4-Pad1): track 0.00 -> 41.2 mm
- net /Analog/R_{out}+: track 23.4 -> 0.00 mm
- net /Analog/L_{out}+: track 23.3 -> 0.00 mm
- net Net-(L2-Pad1): track 51.0 -> 71.6 mm
- net /Digital/ID_SD: track 0.00 -> 17.3 mm
- net Net-(L3-Pad2): track 76.0 -> 91.0 mm
- net Net-(C23-Pad1): track 29.7 -> 41.3 mm
- net Net-(C22-Pad2): track 28.5 -> 40.1 mm
- net Net-(D3-Pad1): track 11.2 -> 0.00 mm
- net /Power/5V: track 128.5 -> 119.3 mm
- net Net-(C32-Pad1): track 8.38 -> 0.00 mm
- net /Digital/ID_SC: track 3.76 -> 11.3 mm
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- added copper zone on B.Cu, net VCC
- removed copper zone on B.Cu, net AVDD
- removed copper zone on F.Cu, net AVDD
- removed copper zone on B.Cu, net DVDD
- removed copper zone on F.Cu, net DVDD

Commit message: WIP
Parts:
- removed D3: ZF16V, Diode_SMD:D_0805_2012Metric
- C32: value 100uF -> 10uF; footprint Capacitor_THT:CP_Radial_D6.3mm_P2.50mm -> Capacitor_SMD:C_0805_2012Metric
- U4, U5: value NCP163 -> NCP163ASN330T1G
- moved C32 14.6 mm to (134.2, 52.9)
- moved C33 13.4 mm to (175.9, 63.9), turned to -45 degrees
- moved R24 13.2 mm to (183.5, 52.1), turned to -90 degrees
- moved R20 11.7 mm to (185.7, 52.1)
- moved R30 10.9 mm to (136.4, 52.9), turned to -90 degrees
- moved R27 8.35 mm to (183.5, 55.7), turned to -90 degrees
- moved J5 7.93 mm to (124.9, 52.9), turned to 90 degrees
- moved R23 7.37 mm to (185.7, 55.7)
- moved C15 6.85 mm to (131.4, 112.9)
- moved C34 4.90 mm to (178.0, 59.8), turned to 0 degrees
- moved C30 4.10 mm to (156.0, 59.8)
- moved C31 1.10 mm to (148.0, 52.7)
- moved C16 0.94 mm to (122.6, 113.0)
- moved R32 0.90 mm to (128.1, 95.3)
- moved L3 0.90 mm to (120.9, 88.1)
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Connections:
- J5 pad 3: Net-(D3-Pad1) -> Net-(C32-Pad1)
Routing:
- net /Analog/MUTE: track 7.06 -> 46.1 mm
- net GND: track 751.3 -> 714.9 mm, vias 72 -> 85
- net VCC: track 162.4 -> 143.4 mm
- net Net-(R20-Pad2): track 33.9 -> 19.3 mm
- net Net-(R23-Pad2): track 25.7 -> 13.6 mm, vias 1 -> 0
- net /Analog/L_{out}+: track 0.00 -> 11.6 mm
- net /Analog/R_{out}+: track 0.00 -> 11.6 mm
- net Net-(L2-Pad1): track 71.6 -> 61.1 mm
- net Net-(C32-Pad1): track 0.00 -> 6.85 mm
- net Net-(L3-Pad2): track 91.0 -> 85.2 mm
- net VEE: track 89.1 -> 94.2 mm, vias 0 -> 1
- net Net-(C22-Pad2): track 40.1 -> 43.5 mm
- added copper zone on F.Cu, net GND
