File: DesktopAMP.kicad_sch (KiCad schematic)
At the start: 2 parts, among them J1 Conn_02x20_Odd_Even, J2 Conn_01x03

Commit message: WIP
Parts:
- added J3: Conn_01x04, Connector_Phoenix_MSTB:PhoenixContact_MSTBVA_2,5_4-G_1x04_P5.00mm_Vertical, symbol Connector_Generic:Conn_01x04
- J1: footprint Etnolit:RPi_Zero_2W -> Etnolit:RPi_Zero_2W_SMD
Connections:
- new net Analog/L_{out}+: J3.3 (Pin_3)
- new net Analog/L_{out}-: J3.4 (Pin_4)
- new net Analog/R_{out}+: J3.2 (Pin_2)
- new net Analog/R_{out}-: J3.1 (Pin_1)
Other:
- sheet Analog ports: added L_{out}+, L_{out}-, R_{out}+, R_{out}-; removed none
- moved on the sheet: J1, J2
