File: analog.kicad_sch (KiCad schematic)
At the start: 27 parts

Commit message: WIP
Parts:
- removed R? (x4): 470R, Resistor_SMD:R_0805_2012Metric, symbol Device:R
- added C23, C24: 1000pF, Capacitor_SMD:C_0805_2012Metric, symbol Device:C
- added R17, R19: 470R, Resistor_SMD:R_0805_2012Metric, symbol Device:R
- R20, R21: renamed from R?; value 470R -> 1K
- gave numbers to parts that had none: 20
Connections:
- net GND: now also C22.1, C25.2, C23.1, C24.1
- net OUTL-: now also R17.2
- net OUTR-: now also R19.2
- net R+: now also J4.4 (Pin_4), R25.2, U7.25
- net at R23.2, R25.1: now also U7.21 (-)
- net at U7.15 (-): now also R22.2, R24.1
- new net: C23.2, R17.1
- new net: C24.2, R19.1
Other:
- moved on the sheet: C22, C25, C26, C27, C28, C29, C30, C31, C32, C33, J4, J5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

Commit message: WIP
Parts:
- removed C22: 1000pF, Capacitor_SMD:C_0805_2012Metric, symbol Device:C
- removed C26, C27: 47uF, Capacitor_THT:CP_Radial_D6.3mm_P2.50mm, symbol Device:C_Polarized
- removed J4: Conn_01x04, Connector_Phoenix_MSTB:PhoenixContact_MSTBVA_2,5_4-G_1x04_P5.00mm_Vertical, symbol Connector_Generic:Conn_01x04
- added C23: 2.2nF, Capacitor_SMD:C_0805_2012Metric, symbol Device:C
- added C32: 100uF, Capacitor_THT:CP_Radial_D6.3mm_P2.50mm, symbol Device:C_Polarized
- added C33: 10uF, Capacitor_THT:CP_Radial_D6.3mm_P2.50mm, symbol Device:C_Polarized
- added C34: 100nF, Capacitor_THT:C_Rect_L7.2mm_W2.5mm_P5.00mm_FKS2_FKP2_MKS2_MKP2, symbol Device:C
- added D3: ZF16V, Diode_SMD:D_0805_2012Metric, symbol Device:D_Zener
- added L2, L3: 0.7uH, Etnolit:L_Axial_L13.25_D11.4_P13.25_Horizontal, symbol Device:L
- added R26, R27: 20K, Resistor_SMD:R_0805_2012Metric, symbol Device:R
- added R28, R29: 3R16, 1W, Resistor_THT:R_Axial_DIN0309_L9.0mm_D3.2mm_P12.70mm_Horizontal, symbol Device:R
- added R31, R32: 10R,3W, Resistor_THT:R_Axial_DIN0617_L17.0mm_D6.0mm_P20.32mm_Horizontal, symbol Device:R
- added R_{load}1, R_{load}2: 8R, symbol Device:R
- C22: renamed from C23; value 1000pF -> 2.2nF
- C24, C25: value 1000pF -> 100nF; footprint Capacitor_SMD:C_0805_2012Metric -> Capacitor_THT:C_Rect_L7.2mm_W2.5mm_P5.00mm_FKS2_FKP2_MKS2_MKP2
- C30: renamed from C32; footprint Capacitor_SMD:C_0805_2012Metric -> Capacitor_THT:C_Rect_L7.2mm_W2.5mm_P5.00mm_FKS2_FKP2_MKS2_MKP2
- C31: renamed from C33; footprint Capacitor_SMD:C_0805_2012Metric -> Capacitor_THT:C_Rect_L7.2mm_W2.5mm_P5.00mm_FKS2_FKP2_MKS2_MKP2
- R21, R22: footprint Resistor_SMD:R_0805_2012Metric -> Resistor_THT:R_Axial_DIN0207_L6.3mm_D2.5mm_P7.62mm_Horizontal
- renumbered C28 to C26, C29 to C27, C30 to C28, C31 to C29, R26 to R30
Connections:
- net GND: now also R24.2, C32.2, C33.2, C34.2, R27.2, R_{load}1.1, R_{load}2.2; no longer C22.1
- net OUTR+: now also R19.2; no longer R18.2
- net OUTR-: now also R18.2; no longer R19.2
- net VCC: now also C33.1, C34.1
- net at R16.1, R20.1: now also C22.2
- net at R17.1: now also C22.1, R21.1; no longer C22.2
- net at R20.2, U7.16 (+): now also R24.1
- net at R22.1: now also R18.1, C23.2
- net at J5.3 (Pin_3): now also D3.1 (K); no longer R30.1
- net at C24.2: now also R28.1; no longer R19.1
- net at R23.1: now also R19.1, C23.1
- net at R21.2: now also R25.1, U7.15 (-); no longer U7.22 (+)
- net L+ renamed L_{out}+
- net L_{out}+: now also R25.2, L2.1, R28.2, R31.2; no longer R24.2
- net R+ renamed R_{out}+
- net R_{out}+: now also L3.2, R26.2, R29.2, R32.1; no longer R25.2
- new net: L2.2, R31.1, R_{load}1.2
- new net: C25.1, R29.1
- new net: R22.2, R26.1, U7.21 (-)
- new net: L3.1, R32.2, R_{load}2.1
- new net: C32.1, D3.2 (A), R30.1
- new net: R23.2, R27.1, U7.22 (+)
Other:
- note added: "L2,L3: Air wound inductor. 1.2mm dia wire, 11 turns around 9mm core"
- note added: "Mute delay circuit"
- note added: "Not on PCB!"
- note added: "Thiel network"
- note added: "Zobel filter"
- moved on the sheet: C22, C26, C27, C28, C29, C30, C31, J5, R16, R17, R24, R30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

Commit message: WIP
Parts:
- L2, L3, R31, R32: now in the parts list
Connections:
- net L_{out}+: now also L2.2, R31.1, R_{load}1.2; no longer L2.1, R25.2, R28.2, R31.2, U7.7
- net R_{out}+: now also L3.1, R32.2, R_{load}2.1; no longer L3.2, R26.2, R29.2, R32.1, U7.25
- new net: L2.1, R25.2, R28.2, R31.2, U7.7
- new net: L3.2, R26.2, R29.2, R32.1, U7.25
Changed lines of the file:
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@@
 (kicad_sch (version 20211123) (generator eeschema)
   (paper "A4")
+  (junction (at 161.29 118.11) (diameter 0) (color 0 0 0 0)
+  )
   (junction (at 214.63 85.09) (diameter 0) (color 0 0 0 0)
   )
@@
   (junction (at 87.63 134.62) (diameter 0) (color 0 0 0 0)
   )
-  (junction (at 161.29 99.06) (diameter 0) (color 0 0 0 0)
-  )
   (junction (at 245.11 85.09) (diameter 0) (color 0 0 0 0)
   )
@@
   (junction (at 161.29 114.3) (diameter 0) (color 0 0 0 0)
   )
+  (junction (at 161.29 54.61) (diameter 0) (color 0 0 0 0)
+  )
   (junction (at 87.63 73.66) (diameter 0) (color 0 0 0 0)
   )
@@
   (junction (at 113.03 99.06) (diameter 0) (color 0 0 0 0)
   )
-  (junction (at 161.29 73.66) (diameter 0) (color 0 0 0 0)
-  )
   (junction (at 229.87 85.09) (diameter 0) (color 0 0 0 0)
   )
@@
     (stroke (width 0) (type default) (color 0 0 0 0))
   )
-  (wire (pts (xy 161.29 52.07) (xy 161.29 58.42))
+  (wire (pts (xy 161.29 52.07) (xy 161.29 54.61))
     (stroke (width 0) (type default) (color 0 0 0 0))
   )
@@
     (stroke (width 0) (type default) (color 0 0 0 0))
   )
-  (wire (pts (xy 161.29 99.06) (xy 177.8 99.06))
+  (wire (pts (xy 161.29 118.11) (xy 177.8 118.11))
     (stroke (width 0) (type default) (color 0 0 0 0))
   )
@@
     (stroke (width 0) (type default) (color 0 0 0 0))
   )
-  (wire (pts (xy 161.29 114.3) (xy 161.29 120.65))
+  (wire (pts (xy 161.29 114.3) (xy 161.29 118.11))
     (stroke (width 0) (type default) (color 0 0 0 0))
   )
@@
     (stroke (width 0) (type default) (color 0 0 0 0))
   )
-  (wire (pts (xy 161.29 73.66) (xy 177.8 73.66))
+  (wire (pts (xy 161.29 54.61) (xy 177.8 54.61))
     (stroke (width 0) (type default) (color 0 0 0 0))
   )
@@
     (stroke (width 0) (type default) (color 0 0 0 0))
   )
+  (wire (pts (xy 161.29 54.61) (xy 161.29 58.42))
+    (stroke (width 0) (type default) (color 0 0 0 0))
+  )
   (wire (pts (xy 97.79 63.5) (xy 97.79 66.04))
+    (stroke (width 0) (type default) (color 0 0 0 0))
+  )
+  (wire (pts (xy 161.29 118.11) (xy 161.29 120.65))
     (stroke (width 0) (type default) (color 0 0 0 0))
   )
@@
     (effects (font (size 1.27 1.27)) (justify left))
   )
-  (hierarchical_label "L_{out}+" (shape output) (at 177.8 73.66 0)
+  (hierarchical_label "L_{out}+" (shape output) (at 177.8 54.61 0)
     (effects (font (size 1.27 1.27)) (justify left))
   )
@@
     (effects (font (size 1.27 1.27)) (justify right))
   )
-  (hierarchical_label "R_{out}+" (shape output) (at 177.8 99.06 0)
+  (hierarchical_label "R_{out}+" (shape output) (at 177.8 118.11 0)
     (effects (font (size 1.27 1.27)) (justify left))
   )
@@
   )
   (symbol (lib_id "Device:L") (at 161.29 64.77 180) (unit 1)
-    (in_bom no) (on_board no) (fields_autoplaced)
+    (in_bom yes) (on_board yes) (fields_autoplaced)
     (property "Reference" "L2" (id 0) (at 162.56 63.4999 0)
       (effects (font (size 1.27 1.27)) (justify right))
@@
   )
   (symbol (lib_id "Device:L") (at 161.29 107.95 180) (unit 1)
-    (in_bom no) (on_board no) (fields_autoplaced)
+    (in_bom yes) (on_board yes) (fields_autoplaced)
     (property "Reference" "L3" (id 0) (at 162.56 106.6799 0)
       (effects (font (size 1.27 1.27)) (justify right))
@@
   )
   (symbol (lib_id "Device:R") (at 149.86 107.95 0) (mirror y) (unit 1)
-    (in_bom no) (on_board no) (fields_autoplaced)
+    (in_bom yes) (on_board yes) (fields_autoplaced)
     (property "Reference" "R32" (id 0) (at 152.4 106.6799 0)
       (effects (font (size 1.27 1.27)) (justify right))
@@
     (pin "1")
   )
-  (symbol (lib_id "Etnolit:LM4780") (at 96.52 116.84 0) (mirror x) (unit 2)
-    (in_bom yes) (on_board yes)
-    (property "Reference" "U7" (id 0) (at 104.14 123.19 0))
-    (property "Value" "LM4780" (id 1) (at 104.14 120.65 0))
+  (symbol (lib_name "LM4780_1") (lib_id "Etnolit:LM4780") (at 96.52 116.84 0) (mirror x) (unit 2)
+    (in_bom yes) (on_board yes)
+    (property "Reference" "U7" (id 0) (at 104.14 110.49 0))
+    (property "Value" "LM4780" (id 1) (at 104.14 113.03 0))
     (property "Footprint" "Etnolit:TO-220-27" (id 2) (at 96.52 116.84 0)
       (effects (font (size 1.27 1.27)) hide)
@@
   )
   (symbol (lib_id "Device:R") (at 149.86 64.77 0) (unit 1)
-    (in_bom no) (on_board no) (fields_autoplaced)
+    (in_bom yes) (on_board yes) (fields_autoplaced)
     (property "Reference" "R31" (id 0) (at 152.4 63.4999 0)
       (effects (font (size 1.27 1.27)) (justify left))

Commit message: WIP
Parts:
- removed C32: 100uF, Capacitor_THT:CP_Radial_D6.3mm_P2.50mm, symbol Device:C_Polarized
- removed D3: ZF16V, Diode_SMD:D_0805_2012Metric, symbol Device:D_Zener
- added C32: 10uF, Capacitor_SMD:C_0805_2012Metric, symbol Device:C
Connections:
- net GND: now also C32.2
- net at J5.3 (Pin_3): now also R30.1, C32.1
Other:
- note removed: "Not on PCB!"
- moved on the sheet: R30
Changed lines of the file:
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@@
   (junction (at 58.42 73.66) (diameter 0) (color 0 0 0 0)
   )
-  (junction (at 259.08 41.91) (diameter 0) (color 0 0 0 0)
+  (junction (at 259.08 39.37) (diameter 0) (color 0 0 0 0)
   )
   (junction (at 87.63 99.06) (diameter 0) (color 0 0 0 0)
@@
     (stroke (width 0) (type default) (color 0 0 0 0))
   )
-  (wire (pts (xy 259.08 41.91) (xy 259.08 44.45))
+  (wire (pts (xy 259.08 39.37) (xy 259.08 41.91))
     (stroke (width 0) (type default) (color 0 0 0 0))
   )
@@
     (stroke (width 0) (type default) (color 0 0 0 0))
   )
-  (wire (pts (xy 259.08 29.21) (xy 259.08 31.75))
-    (stroke (width 0) (type default) (color 0 0 0 0))
-  )
   (wire (pts (xy 38.1 99.06) (xy 41.91 99.06))
     (stroke (width 0) (type default) (color 0 0 0 0))
   )
-  (wire (pts (xy 271.78 44.45) (xy 271.78 41.91))
+  (wire (pts (xy 271.78 41.91) (xy 271.78 39.37))
     (stroke (width 0) (type default) (color 0 0 0 0))
   )
@@
     (stroke (width 0) (type default) (color 0 0 0 0))
   )
-  (wire (pts (xy 259.08 39.37) (xy 259.08 41.91))
+  (wire (pts (xy 259.08 29.21) (xy 259.08 39.37))
     (stroke (width 0) (type default) (color 0 0 0 0))
   )
@@
     (stroke (width 0) (type default) (color 0 0 0 0))
   )
-  (wire (pts (xy 271.78 41.91) (xy 259.08 41.91))
+  (wire (pts (xy 271.78 39.37) (xy 259.08 39.37))
     (stroke (width 0) (type default) (color 0 0 0 0))
   )
@@
     (stroke (width 0) (type default) (color 0 0 0 0))
   )
-  (wire (pts (xy 271.78 52.07) (xy 271.78 54.61))
-    (stroke (width 0) (type default) (color 0 0 0 0))
-  )
-  (wire (pts (xy 259.08 52.07) (xy 259.08 54.61))
+  (wire (pts (xy 271.78 49.53) (xy 271.78 52.07))
+    (stroke (width 0) (type default) (color 0 0 0 0))
+  )
+  (wire (pts (xy 259.08 49.53) (xy 259.08 52.07))
     (stroke (width 0) (type default) (color 0 0 0 0))
   )
@@
   )
   (text "Zobel filter" (at 124.46 87.63 0)
-    (effects (font (size 1.27 1.27)) (justify left bottom))
-  )
-  (text "Not on PCB!" (at 146.05 33.02 0)
     (effects (font (size 1.27 1.27)) (justify left bottom))
   )
@@
     (pin "9")
   )
-  (symbol (lib_id "power:GND") (at 271.78 54.61 0) (unit 1)
-    (in_bom yes) (on_board yes)
-    (property "Reference" "#PWR055" (id 0) (at 271.78 60.96 0)
-      (effects (font (size 1.27 1.27)) hide)
-    )
-    (property "Value" "GND" (id 1) (at 271.78 59.69 0)
-      (effects (font (size 1.27 1.27)) hide)
-    )
-    (property "Footprint" "" (id 2) (at 271.78 54.61 0)
-      (effects (font (size 1.27 1.27)) hide)
-    )
-    (property "Datasheet" "" (id 3) (at 271.78 54.61 0)
+  (symbol (lib_id "power:GND") (at 271.78 52.07 0) (unit 1)
+    (in_bom yes) (on_board yes)
+    (property "Reference" "#PWR055" (id 0) (at 271.78 58.42 0)
+      (effects (font (size 1.27 1.27)) hide)
+    )
+    (property "Value" "GND" (id 1) (at 271.78 57.15 0)
+      (effects (font (size 1.27 1.27)) hide)
+    )
+    (property "Footprint" "" (id 2) (at 271.78 52.07 0)
+      (effects (font (size 1.27 1.27)) hide)
+    )
+    (property "Datasheet" "" (id 3) (at 271.78 52.07 0)
       (effects (font (size 1.27 1.27)) hide)
     )
@@
     (pin "1")
   )
-  (symbol (lib_id "power:VEE") (at 259.08 54.61 180) (unit 1)
-    (in_bom yes) (on_board yes) (fields_autoplaced)
-    (property "Reference" "#PWR054" (id 0) (at 259.08 50.8 0)
-      (effects (font (size 1.27 1.27)) hide)
-    )
-    (property "Value" "VEE" (id 1) (at 259.08 59.69 0))
-    (property "Footprint" "" (id 2) (at 259.08 54.61 0)
-      (effects (font (size 1.27 1.27)) hide)
-    )
-    (property "Datasheet" "" (id 3) (at 259.08 54.61 0)
+  (symbol (lib_id "power:VEE") (at 259.08 52.07 180) (unit 1)
+    (in_bom yes) (on_board yes) (fields_autoplaced)
+    (property "Reference" "#PWR054" (id 0) (at 259.08 48.26 0)
+      (effects (font (size 1.27 1.27)) hide)
+    )
+    (property "Value" "VEE" (id 1) (at 259.08 57.15 0))
+    (property "Footprint" "" (id 2) (at 259.08 52.07 0)
+      (effects (font (size 1.27 1.27)) hide)
+    )
+    (property "Datasheet" "" (id 3) (at 259.08 52.07 0)
       (effects (font (size 1.27 1.27)) hide)
     )
@@
     (pin "2")
   )
-  (symbol (lib_id "Device:C_Polarized") (at 271.78 48.26 0) (unit 1)
-    (in_bom yes) (on_board yes) (fields_autoplaced)
-    (property "Reference" "C32" (id 0) (at 275.59 46.1009 0)
-      (effects (font (size 1.27 1.27)) (justify left))
-    )
-    (property "Value" "100uF" (id 1) (at 275.59 48.6409 0)
-      (effects (font (size 1.27 1.27)) (justify left))
-    )
-    (property "Footprint" "Capacitor_THT:CP_Radial_D6.3mm_P2.50mm" (id 2) (at 272.7452 52.07 0)
-      (effects (font (size 1.27 1.27)) hide)
-    )
-    (property "Datasheet" "~" (id 3) (at 271.78 48.26 0)
-      (effects (font (size 1.27 1.27)) hide)
-    )
-    (pin "1")
-    (pin "2")
-  )
   (symbol (lib_id "power:VEE") (at 229.87 99.06 180) (unit 1)
     (in_bom yes) (on_board yes)
@@
     (pin "1")
   )
-  (symbol (lib_id "Device:R") (at 259.08 48.26 0) (unit 1)
-    (in_bom yes) (on_board yes) (fields_autoplaced)
-    (property "Reference" "R30" (id 0) (at 261.62 46.9899 0)
-      (effects (font (size 1.27 1.27)) (justify left))
-    )
-    (property "Value" "10K" (id 1) (at 261.62 49.5299 0)
-      (effects (font (size 1.27 1.27)) (justify left))
-    )
-    (property "Footprint" "Resistor_SMD:R_0805_2012Metric" (id 2) (at 257.302 48.26 90)
-      (effects (font (size 1.27 1.27)) hide)
-    )
-    (property "Datasheet" "~" (id 3) (at 259.08 48.26 0)
+  (symbol (lib_id "Device:R") (at 259.08 45.72 0) (unit 1)
+    (in_bom yes) (on_board yes) (fields_autoplaced)
+    (property "Reference" "R30" (id 0) (at 261.62 44.4499 0)
+      (effects (font (size 1.27 1.27)) (justify left))
+    )
+    (property "Value" "10K" (id 1) (at 261.62 46.9899 0)
+      (effects (font (size 1.27 1.27)) (justify left))
+    )
+    (property "Footprint" "Resistor_SMD:R_0805_2012Metric" (id 2) (at 257.302 45.72 90)
+      (effects (font (size 1.27 1.27)) hide)
+    )
+    (property "Datasheet" "~" (id 3) (at 259.08 45.72 0)
       (effects (font (size 1.27 1.27)) hide)
     )
@@
     (pin "2")
   )
+  (symbol (lib_id "Device:C") (at 271.78 45.72 0) (unit 1)
+    (in_bom yes) (on_board yes) (fields_autoplaced)
+    (property "Reference" "C32" (id 0) (at 275.59 44.4499 0)
+      (effects (font (size 1.27 1.27)) (justify left))
+    )
+    (property "Value" "10uF" (id 1) (at 275.59 46.9899 0)
+      (effects (font (size 1.27 1.27)) (justify left))
+    )
+    (property "Footprint" "Capacitor_SMD:C_0805_2012Metric" (id 2) (at 272.7452 49.53 0)
+      (effects (font (size 1.27 1.27)) hide)
+    )
+    (property "Datasheet" "~" (id 3) (at 271.78 45.72 0)
+      (effects (font (size 1.27 1.27)) hide)
+    )
+    (pin "1")
+    (pin "2")
+  )
   (symbol (lib_id "Device:C_Polarized") (at 214.63 76.2 0) (unit 1)
     (in_bom yes) (on_board yes) (fields_autoplaced)
@@
   (symbol (lib_name "LM4780_1") (lib_id "Etnolit:LM4780") (at 96.52 116.84 0) (mirror x) (unit 2)
     (in_bom yes) (on_board yes)
-    (property "Reference" "U7" (id 0) (at 104.14 110.49 0))
-    (property "Value" "LM4780" (id 1) (at 104.14 113.03 0))
+    (property "Reference" "U7" (id 0) (at 104.14 123.19 0))
+    (property "Value" "LM4780" (id 1) (at 104.14 120.65 0))
     (property "Footprint" "Etnolit:TO-220-27" (id 2) (at 96.52 116.84 0)
       (effects (font (size 1.27 1.27)) hide)
@@
     (pin "25")
   )
-  (symbol (lib_id "Device:D_Zener") (at 259.08 35.56 270) (unit 1)
-    (in_bom yes) (on_board yes) (fields_autoplaced)
-    (property "Reference" "D3" (id 0) (at 261.62 34.2899 90)
-      (effects (font (size 1.27 1.27)) (justify left))
-    )
-    (property "Value" "ZF16V" (id 1) (at 261.62 36.8299 90)
-      (effects (font (size 1.27 1.27)) (justify left))
-    )
-    (property "Footprint" "Diode_SMD:D_0805_2012Metric" (id 2) (at 259.08 35.56 0)
-      (effects (font (size 1.27 1.27)) hide)
-    )
-    (property "Datasheet" "~" (id 3) (at 259.08 35.56 0)
-      (effects (font (size 1.27 1.27)) hide)
-    )
-    (pin "1")
-    (pin "2")
-  )
   (symbol (lib_id "power:GND") (at 175.26 137.16 0) (unit 1)
